File: AttinySwitch/AttinySwitch.sch (KiCad schematic (older format))
At the start: 4 parts, among them IC1 ATTINY84-P, K1 CONN_3, P1 CONN_4X2

Commit message: Added voltage regulator and SSR
Parts:
- added P2: PWR/LOAD, symbol PWR/LOAD
- added P?: CONN_2, symbol CONN_2
- added Q1: 2N3904, TO92, symbol PN2222A
- added R2: 10K, symbol R
- added R3: 1K, symbol R
- added U1: AQH3223, symbol AQH3223
Connections:
- wire segments 42 -> 63
Changed lines of the file:
@@
 LIBS:valves
 LIBS:AttinySwitch-cache
-EELAYER 24 0
+EELAYER 27 0
 EELAYER END
 $Descr A4 11693 8268
@@
 Sheet 1 1
 Title ""
-Date ""
+Date "17 feb 2014"
 Rev ""
 Comp ""
@@
 	1    0    0    -1
 $EndComp
+$Comp
+L PN2222A Q1
+U 1 1 53027A15
+P 6500 1550
+F 0 "Q1" H 6500 1402 40  0000 R CNN
+F 1 "2N3904" H 6500 1700 40  0000 R CNN
+F 2 "TO92" H 6400 1652 29  0000 C CNN
+F 3 "~" H 6500 1550 60  0000 C CNN
+	1    6500 1550
+	0    1    -1   0
+$EndComp
+$Comp
+L R R2
+U 1 1 53027A4B
+P 5750 1950
+F 0 "R2" V 5650 1950 40  0000 C CNN
+F 1 "10K" V 5750 1950 40  0000 C CNN
+F 2 "" V 5680 1950 30  0000 C CNN
+F 3 "" H 5750 1950 30  0000 C CNN
+	1    5750 1950
+	0    -1   -1   0
+$EndComp
+$Comp
+L R R3
+U 1 1 53027A55
+P 7100 1700
+F 0 "R3" V 7180 1700 40  0000 C CNN
+F 1 "1K" V 7107 1701 40  0000 C CNN
+F 2 "" V 7030 1700 30  0000 C CNN
+F 3 "" H 7100 1700 30  0000 C CNN
+	1    7100 1700
+	1    0    0    -1
+$EndComp
+$Comp
+L AQH3223 U1
+U 1 1 53028552
+P 8350 1700
+F 0 "U1" H 8550 2000 60  0000 C CNN
+F 1 "AQH3223" H 8300 1400 60  0000 C CNN
+F 2 "" H 8350 1700 60  0000 C CNN
+F 3 "" H 8350 1700 60  0000 C CNN
+	1    8350 1700
+	1    0    0    -1
+$EndComp
 Wire Wire Line
 	4650 2600 4650 2250
 Wire Wire Line
-	7350 2250 7350 3150
-Wire Wire Line
 	7350 3150 7650 3150
 Wire Wire Line
-	4650 3800 4650 4150
+	4650 3600 4650 4150
 Wire Wire Line
 	2900 4150 7350 4150
@@
 	4500 3250 4500 2250
 Wire Wire Line
-	4500 2250 7350 2250
-Wire Wire Line
 	2900 4150 2900 2950
 Wire Wire Line
@@
 Wire Wire Line
 	4200 3050 4000 3050
+Wire Wire Line
+	7350 1450 7350 3150
+Wire Wire Line
+	6700 1450 7350 1450
+Connection ~ 7100 1450
+Wire Wire Line
+	6500 1750 6500 1950
+Wire Wire Line
+	6000 1950 7700 1950
+Connection ~ 6500 1950
+Wire Wire Line
+	6300 1450 4850 1450
+Wire Wire Line
+	4850 1450 4850 2250
+Wire Wire Line
+	4850 2250 4500 2250
+Wire Wire Line
+	5500 1950 4700 1950
+Wire Wire Line
+	4700 1950 4700 3600
+Wire Wire Line
+	4700 3600 4650 3600
+Connection ~ 4650 3800
+Connection ~ 7100 1950
+Wire Wire Line
+	6750 2700 7250 2700
+Wire Wire Line
+	7250 2700 7250 2100
+Wire Wire Line
+	7250 2100 7600 2100
+Wire Wire Line
+	7600 2100 7600 1500
+Wire Wire Line
+	7600 1500 7700 1500
+Wire Wire Line
+	8950 1600 8950 1500
+Wire Wire Line
+	8950 1900 8950 1700
+$Comp
+L PWR/LOAD P2
+U 1 1 53029832
+P 9500 1750
+F 0 "P2" V 9450 1800 50  0000 C CNN
+F 1 "PWR/LOAD" V 9550 1750 50  0000 C CNN
+F 2 "" H 9500 1750 60  0000 C CNN
+F 3 "" H 9500 1750 60  0000 C CNN
+	1    9500 1750
+	1    0    0    -1
+$EndComp
+Wire Wire Line
+	8950 1600 9150 1600
+Wire Wire Line
+	8950 1700 9150 1700
+$Comp
+L CONN_2 P?
+U 1 1 53029AF5
+P 9500 2400
+F 0 "P?" V 9450 2400 40  0000 C CNN
+F 1 "CONN_2" V 9550 2400 40  0000 C CNN
+F 2 "" H 9500 2400 60  0000 C CNN
+F 3 "" H 9500 2400 60  0000 C CNN
+	1    9500 2400
+	1    0    0    -1
+$EndComp
+Wire Wire Line
+	9150 1800 9000 1800
+Wire Wire Line
+	9000 1800 9000 2300
+Wire Wire Line
+	9000 2300 9150 2300
+Wire Wire Line
+	9150 1900 9150 2500
 $EndSCHEMATC

Commit message: Added switch and wireless interrupt to Pin 5 (INT 0)
Parts:
- added P4: SWITCH, symbol CONN_2
- added R4: 1M, symbol R
- added R5, R6: 100K, symbol R
- gave numbers to parts that had none: 1
Connections:
- wire segments 63 -> 76
Changed lines of the file:
@@
 Sheet 1 1
 Title ""
-Date "17 feb 2014"
+Date "21 feb 2014"
 Rev ""
 Comp ""
@@
 	1    0    0    -1
 $EndComp
-Wire Wire Line
-	4650 2600 4650 2250
-Wire Wire Line
-	7350 3150 7650 3150
-Wire Wire Line
-	4650 3600 4650 4150
-Wire Wire Line
-	2900 4150 7350 4150
-Wire Wire Line
-	7350 4150 7350 3250
-Wire Wire Line
-	7350 3250 7650 3250
-Connection ~ 4650 2250
-Connection ~ 4650 4150
-Wire Wire Line
-	7250 3950 7250 2900
-Wire Wire Line
-	7250 2900 6750 2900
-Wire Wire Line
-	7050 4050 7050 3300
-Wire Wire Line
-	7050 3300 6750 3300
-Wire Wire Line
-	3050 4100 7150 4100
-Wire Wire Line
-	7150 4100 7150 3000
-Wire Wire Line
-	7150 3000 6750 3000
-Wire Wire Line
-	4350 4000 6950 4000
-Wire Wire Line
-	6950 4000 6950 3100
-Wire Wire Line
-	6950 3100 6750 3100
-Wire Wire Line
-	6850 2450 6850 3200
-Wire Wire Line
-	6850 3200 6750 3200
-Wire Wire Line
-	7550 2900 7550 3350
-Wire Wire Line
-	7550 3350 7650 3350
-Wire Wire Line
-	6750 3500 6900 3500
-Wire Wire Line
-	6900 3500 6900 2350
-Wire Wire Line
-	6900 2350 7550 2350
-Wire Wire Line
-	7550 2350 7550 2400
-Wire Wire Line
-	4000 3250 4500 3250
-Wire Wire Line
-	4500 3250 4500 2250
-Wire Wire Line
-	2900 4150 2900 2950
-Wire Wire Line
-	2900 2950 3200 2950
-Wire Wire Line
-	4000 2950 4100 2950
-Wire Wire Line
-	4100 2950 4100 3950
-Connection ~ 4100 3950
-Wire Wire Line
-	4100 3950 7250 3950
-Wire Wire Line
-	7050 4050 3200 4050
-Wire Wire Line
-	3200 4050 3200 3250
-Wire Wire Line
-	3050 4100 3050 3050
-Wire Wire Line
-	3050 3050 3200 3050
-Wire Wire Line
-	4350 4000 4350 3150
-Wire Wire Line
-	4350 3150 4000 3150
-Wire Wire Line
-	6850 2450 4200 2450
-Wire Wire Line
-	4200 2450 4200 3050
-Wire Wire Line
-	4200 3050 4000 3050
-Wire Wire Line
-	7350 1450 7350 3150
-Wire Wire Line
-	6700 1450 7350 1450
-Connection ~ 7100 1450
-Wire Wire Line
-	6500 1750 6500 1950
-Wire Wire Line
-	6000 1950 7700 1950
-Connection ~ 6500 1950
-Wire Wire Line
-	6300 1450 4850 1450
-Wire Wire Line
-	4850 1450 4850 2250
-Wire Wire Line
-	4850 2250 4500 2250
-Wire Wire Line
-	5500 1950 4700 1950
-Wire Wire Line
-	4700 1950 4700 3600
-Wire Wire Line
-	4700 3600 4650 3600
-Connection ~ 4650 3800
-Connection ~ 7100 1950
-Wire Wire Line
-	6750 2700 7250 2700
-Wire Wire Line
-	7250 2700 7250 2100
-Wire Wire Line
-	7250 2100 7600 2100
-Wire Wire Line
-	7600 2100 7600 1500
-Wire Wire Line
-	7600 1500 7700 1500
-Wire Wire Line
-	8950 1600 8950 1500
-Wire Wire Line
-	8950 1900 8950 1700
 $Comp
 L PWR/LOAD P2
@@
 	1    0    0    -1
 $EndComp
-Wire Wire Line
-	8950 1600 9150 1600
-Wire Wire Line
-	8950 1700 9150 1700
-$Comp
-L CONN_2 P?
+$Comp
+L CONN_2 P3
 U 1 1 53029AF5
 P 9500 2400
-F 0 "P?" V 9450 2400 40  0000 C CNN
+F 0 "P3" V 9450 2400 40  0000 C CNN
 F 1 "CONN_2" V 9550 2400 40  0000 C CNN
 F 2 "" H 9500 2400 60  0000 C CNN
@@
 	1    0    0    -1
 $EndComp
+$Comp
+L CONN_2 P4
+U 1 1 53073854
+P 9500 2900
+F 0 "P4" V 9450 2900 40  0000 C CNN
+F 1 "SWITCH" V 9550 2900 40  0000 C CNN
+F 2 "" H 9500 2900 60  0000 C CNN
+F 3 "" H 9500 2900 60  0000 C CNN
+	1    9500 2900
+	1    0    0    -1
+$EndComp
+$Comp
+L R R4
+U 1 1 53073982
+P 8050 2800
+F 0 "R4" V 8130 2800 40  0000 C CNN
+F 1 "1M" V 8057 2801 40  0000 C CNN
+F 2 "" V 7980 2800 30  0000 C CNN
+F 3 "" H 8050 2800 30  0000 C CNN
+	1    8050 2800
+	0    -1   -1   0
+$EndComp
+$Comp
+L R R5
+U 1 1 53073988
+P 8700 2800
+F 0 "R5" V 8780 2800 40  0000 C CNN
+F 1 "100K" V 8707 2801 40  0000 C CNN
+F 2 "" V 8630 2800 30  0000 C CNN
+F 3 "" H 8700 2800 30  0000 C CNN
+	1    8700 2800
+	0    -1   -1   0
+$EndComp
+$Comp
+L R R6
+U 1 1 5307398E
+P 8700 3000
+F 0 "R6" V 8780 3000 40  0000 C CNN
+F 1 "100K" V 8707 3001 40  0000 C CNN
+F 2 "" V 8630 3000 30  0000 C CNN
+F 3 "" H 8700 3000 30  0000 C CNN
+	1    8700 3000
+	0    -1   -1   0
+$EndComp
+Wire Wire Line
+	4650 2600 4650 2250
+Wire Wire Line
+	7350 3150 7650 3150
+Wire Wire Line
+	4650 3600 4650 4150
+Wire Wire Line
+	2900 4150 8450 4150
+Wire Wire Line
+	7350 4150 7350 3250
+Wire Wire Line
+	7350 3250 7650 3250
+Connection ~ 4650 2250
+Connection ~ 4650 4150
+Wire Wire Line
+	7250 3950 7250 2900
+Wire Wire Line
+	7250 2900 6750 2900
+Wire Wire Line
+	7050 4050 7050 3300
+Wire Wire Line
+	7050 3300 6750 3300
+Wire Wire Line
+	3050 4100 7150 4100
+Wire Wire Line
+	7150 4100 7150 3000
+Wire Wire Line
+	7150 3000 6750 3000
+Wire Wire Line
+	4350 4000 6950 4000
+Wire Wire Line
+	6950 4000 6950 3100
+Wire Wire Line
+	6950 3100 6750 3100
+Wire Wire Line
+	6850 2450 6850 3200
+Wire Wire Line
+	6850 3200 6750 3200
+Wire Wire Line
+	7550 2900 7550 3350
+Wire Wire Line
+	7550 3350 7650 3350
+Wire Wire Line
+	6750 3500 6900 3500
+Wire Wire Line
+	6900 3500 6900 2350
+Wire Wire Line
+	6900 2350 7550 2350
+Wire Wire Line
+	7550 2350 7550 2400
+Wire Wire Line
+	4000 3250 4500 3250
+Wire Wire Line
+	4500 3250 4500 2250
+Wire Wire Line
+	2900 4150 2900 2950
+Wire Wire Line
+	2900 2950 3200 2950
+Wire Wire Line
+	4000 2950 4100 2950
+Wire Wire Line
+	4100 2950 4100 3950
+Connection ~ 4100 3950
+Wire Wire Line
+	4100 3950 7250 3950
+Wire Wire Line
+	7050 4050 3200 4050
+Wire Wire Line
+	3200 4050 3200 3250
+Wire Wire Line
+	3050 4100 3050 3050
+Wire Wire Line
+	3050 3050 3200 3050
+Wire Wire Line
+	4350 4000 4350 3150
+Wire Wire Line
+	4350 3150 4000 3150
+Wire Wire Line
+	6850 2450 4200 2450
+Wire Wire Line
+	4200 2450 4200 3050
+Wire Wire Line
+	4200 3050 4000 3050
+Wire Wire Line
+	7350 1450 7350 3150
+Wire Wire Line
+	6700 1450 7350 1450
+Connection ~ 7100 1450
+Wire Wire Line
+	6500 1750 6500 1950
+Wire Wire Line
+	6000 1950 7700 1950
+Connection ~ 6500 1950
+Wire Wire Line
+	6300 1450 4850 1450
+Wire Wire Line
+	4850 1450 4850 2250
+Wire Wire Line
+	4500 2250 7800 2250
+Wire Wire Line
+	5500 1950 4700 1950
+Wire Wire Line
+	4700 1950 4700 3600
+Wire Wire Line
+	4700 3600 4650 3600
+Connection ~ 4650 3800
+Connection ~ 7100 1950
+Wire Wire Line
+	6750 2700 7250 2700
+Wire Wire Line
+	7250 2700 7250 2100
+Wire Wire Line
+	7250 2100 7600 2100
+Wire Wire Line
+	7600 2100 7600 1500
+Wire Wire Line
+	7600 1500 7700 1500
+Wire Wire Line
+	8950 1600 8950 1500
+Wire Wire Line
+	8950 1900 8950 1700
+Wire Wire Line
+	8950 1600 9150 1600
+Wire Wire Line
+	8950 1700 9150 1700
 Wire Wire Line
 	9150 1800 9000 1800
@@
 Wire Wire Line
 	9150 1900 9150 2500
+Wire Wire Line
+	6750 2200 8350 2200
+Wire Wire Line
+	6750 2200 6750 2600
+Wire Wire Line
+	8300 2800 8450 2800
+Wire Wire Line
+	8350 2200 8350 2800
+Connection ~ 8350 2800
+Wire Wire Line
+	8950 2800 9150 2800
+Wire Wire Line
+	7800 2250 7800 2800
+Connection ~ 4850 2250
+Wire Wire Line
+	9150 3000 8950 3000
+Wire Wire Line
+	8450 4150 8450 3000
+Connection ~ 7350 4150
+Wire Wire Line
+	3200 3150 3150 3150
+Wire Wire Line
+	3150 3150 3150 4300
+Wire Wire Line
+	3150 4300 6900 4300
+Wire Wire Line
+	6900 4300 6900 3700
+Wire Wire Line
+	6900 3700 6750 3700
 $EndSCHEMATC

Commit message: Added push button to interrupt pin
Parts:
- removed R5: 100K, symbol R
- added D1: LED, ~, symbol LED
- Q1: value 2N3904 -> PN2222A
- R4: value 1M -> 220
Connections:
- net labels added: +5v, GND, Serial out
- wire segments 76 -> 73
Other:
- moved on the sheet: R6
Changed lines of the file:
@@
 Sheet 1 1
 Title ""
-Date "21 feb 2014"
+Date "1 mar 2014"
 Rev ""
 Comp ""
@@
 	1    7550 2650
 	1    0    0    -1
-$EndComp
-$Comp
-L PN2222A Q1
-U 1 1 53027A15
-P 6500 1550
-F 0 "Q1" H 6500 1402 40  0000 R CNN
-F 1 "2N3904" H 6500 1700 40  0000 R CNN
-F 2 "TO92" H 6400 1652 29  0000 C CNN
-F 3 "~" H 6500 1550 60  0000 C CNN
-	1    6500 1550
-	0    1    -1   0
 $EndComp
 $Comp
@@
 $EndComp
 $Comp
-L R R4
-U 1 1 53073982
-P 8050 2800
-F 0 "R4" V 8130 2800 40  0000 C CNN
-F 1 "1M" V 8057 2801 40  0000 C CNN
-F 2 "" V 7980 2800 30  0000 C CNN
-F 3 "" H 8050 2800 30  0000 C CNN
-	1    8050 2800
-	0    -1   -1   0
-$EndComp
-$Comp
-L R R5
-U 1 1 53073988
-P 8700 2800
-F 0 "R5" V 8780 2800 40  0000 C CNN
-F 1 "100K" V 8707 2801 40  0000 C CNN
-F 2 "" V 8630 2800 30  0000 C CNN
-F 3 "" H 8700 2800 30  0000 C CNN
-	1    8700 2800
-	0    -1   -1   0
-$EndComp
-$Comp
 L R R6
 U 1 1 5307398E
-P 8700 3000
-F 0 "R6" V 8780 3000 40  0000 C CNN
-F 1 "100K" V 8707 3001 40  0000 C CNN
-F 2 "" V 8630 3000 30  0000 C CNN
-F 3 "" H 8700 3000 30  0000 C CNN
-	1    8700 3000
+P 8450 3900
+F 0 "R6" V 8530 3900 40  0000 C CNN
+F 1 "100K" V 8457 3901 40  0000 C CNN
+F 2 "" V 8380 3900 30  0000 C CNN
+F 3 "" H 8450 3900 30  0000 C CNN
+	1    8450 3900
+	-1   0    0    1
+$EndComp
+Text Label 7600 3150 0    39   ~ 0
++5v
+Text Label 7600 3250 0    39   ~ 0
+GND
+Text Label 7550 3450 0    39   ~ 0
+Serial out
+Wire Wire Line
+	6750 3700 7650 3700
+Wire Wire Line
+	8450 2250 8450 2800
+Wire Wire Line
+	3200 3150 3150 3150
+Connection ~ 7350 4150
+Wire Wire Line
+	8450 3000 9150 3000
+Connection ~ 4850 2250
+Wire Wire Line
+	8450 2800 9150 2800
+Wire Wire Line
+	9150 1900 9150 2500
+Wire Wire Line
+	9000 2300 9150 2300
+Wire Wire Line
+	9000 1800 9000 2300
+Wire Wire Line
+	9150 1800 9000 1800
+Wire Wire Line
+	8950 1700 9150 1700
+Wire Wire Line
+	8950 1600 9150 1600
+Wire Wire Line
+	8950 1900 8950 1700
+Wire Wire Line
+	8950 1600 8950 1500
+Wire Wire Line
+	7600 1500 7700 1500
+Wire Wire Line
+	7600 2100 7600 1500
+Wire Wire Line
+	7250 2100 8800 2100
+Wire Wire Line
+	7250 2700 7250 2100
+Wire Wire Line
+	6750 2700 7250 2700
+Connection ~ 7100 1950
+Connection ~ 4650 3800
+Wire Wire Line
+	4700 3600 4650 3600
+Wire Wire Line
+	4700 1950 4700 3600
+Wire Wire Line
+	5500 1950 4700 1950
+Wire Wire Line
+	4500 2250 8450 2250
+Wire Wire Line
+	4850 1450 4850 2250
+Wire Wire Line
+	6300 1450 4850 1450
+Connection ~ 6500 1950
+Wire Wire Line
+	6000 1950 7700 1950
+Wire Wire Line
+	6500 1750 6500 1950
+Connection ~ 7100 1450
+Wire Wire Line
+	6700 1450 7350 1450
+Wire Wire Line
+	7350 1450 7350 3150
+Wire Wire Line
+	4200 3050 4000 3050
+Wire Wire Line
+	4200 2450 4200 3050
+Wire Wire Line
+	6850 2450 4200 2450
+Wire Wire Line
+	4350 3150 4000 3150
+Wire Wire Line
+	4350 4000 4350 3150
+Wire Wire Line
+	3050 3050 3200 3050
+Wire Wire Line
+	3050 4100 3050 3050
+Wire Wire Line
+	3200 4050 3200 3250
+Wire Wire Line
+	7050 4050 3200 4050
+Wire Wire Line
+	4100 3950 7250 3950
+Connection ~ 4100 3950
+Wire Wire Line
+	4100 2950 4100 3950
+Wire Wire Line
+	4000 2950 4100 2950
+Wire Wire Line
+	2900 2950 3200 2950
+Wire Wire Line
+	2900 4150 2900 2950
+Wire Wire Line
+	4500 3250 4500 2250
+Wire Wire Line
+	4000 3250 4500 3250
+Wire Wire Line
+	7550 2350 7550 2400
+Wire Wire Line
+	6900 2350 7550 2350
+Wire Wire Line
+	6900 3500 6900 2350
+Wire Wire Line
+	6750 3500 6900 3500
+Wire Wire Line
+	7550 3350 7650 3350
+Wire Wire Line
+	7550 2900 7550 3350
+Wire Wire Line
+	6850 3200 6750 3200
+Wire Wire Line
+	6850 2450 6850 3200
+Wire Wire Line
+	6950 3100 6750 3100
+Wire Wire Line
+	6950 4000 6950 3100
+Wire Wire Line
+	4350 4000 6950 4000
+Wire Wire Line
+	7150 3000 6750 3000
+Wire Wire Line
+	7150 4100 7150 3000
+Wire Wire Line
+	3050 4100 7150 4100
+Wire Wire Line
+	7050 3300 6750 3300
+Wire Wire Line
+	7050 4050 7050 3300
+Wire Wire Line
+	7250 2900 6750 2900
+Wire Wire Line
+	7250 3950 7250 2900
+Connection ~ 4650 4150
+Connection ~ 4650 2250
+Wire Wire Line
+	7350 3250 7650 3250
+Wire Wire Line
+	7350 4150 7350 3250
+Wire Wire Line
+	2900 4150 9300 4150
+Wire Wire Line
+	4650 3600 4650 4150
+Wire Wire Line
+	7350 3150 7650 3150
+Wire Wire Line
+	4650 2600 4650 2250
+Wire Wire Line
+	7650 3700 7650 3650
+Wire Wire Line
+	7650 3650 8450 3650
+Wire Wire Line
+	8450 3650 8450 3000
+$Comp
+L LED D1
+U 1 1 5311FE82
+P 9300 3950
+F 0 "D1" H 9300 4050 50  0000 C CNN
+F 1 "LED" H 9300 3850 50  0000 C CNN
+F 2 "~" H 9300 3950 60  0000 C CNN
+F 3 "~" H 9300 3950 60  0000 C CNN
+	1    9300 3950
+	0    1    1    0
+$EndComp
+$Comp
+L R R4
+U 1 1 5311FE8F
+P 9050 3500
+F 0 "R4" V 9130 3500 40  0000 C CNN
+F 1 "220" V 9057 3501 40  0000 C CNN
+F 2 "" V 8980 3500 30  0000 C CNN
+F 3 "" H 9050 3500 30  0000 C CNN
+	1    9050 3500
 	0    -1   -1   0
 $EndComp
 Wire Wire Line
-	4650 2600 4650 2250
-Wire Wire Line
-	7350 3150 7650 3150
-Wire Wire Line
-	4650 3600 4650 4150
-Wire Wire Line
-	2900 4150 8450 4150
-Wire Wire Line
-	7350 4150 7350 3250
-Wire Wire Line
-	7350 3250 7650 3250
-Connection ~ 4650 2250
-Connection ~ 4650 4150
-Wire Wire Line
-	7250 3950 7250 2900
-Wire Wire Line
-	7250 2900 6750 2900
-Wire Wire Line
-	7050 4050 7050 3300
-Wire Wire Line
-	7050 3300 6750 3300
-Wire Wire Line
-	3050 4100 7150 4100
-Wire Wire Line
-	7150 4100 7150 3000
-Wire Wire Line
-	7150 3000 6750 3000
-Wire Wire Line
-	4350 4000 6950 4000
-Wire Wire Line
-	6950 4000 6950 3100
-Wire Wire Line
-	6950 3100 6750 3100
-Wire Wire Line
-	6850 2450 6850 3200
-Wire Wire Line
-	6850 3200 6750 3200
-Wire Wire Line
-	7550 2900 7550 3350
-Wire Wire Line
-	7550 3350 7650 3350
-Wire Wire Line
-	6750 3500 6900 3500
-Wire Wire Line
-	6900 3500 6900 2350
-Wire Wire Line
-	6900 2350 7550 2350
-Wire Wire Line
-	7550 2350 7550 2400
-Wire Wire Line
-	4000 3250 4500 3250
-Wire Wire Line
-	4500 3250 4500 2250
-Wire Wire Line
-	2900 4150 2900 2950
-Wire Wire Line
-	2900 2950 3200 2950
-Wire Wire Line
-	4000 2950 4100 2950
-Wire Wire Line
-	4100 2950 4100 3950
-Connection ~ 4100 3950
-Wire Wire Line
-	4100 3950 7250 3950
-Wire Wire Line
-	7050 4050 3200 4050
-Wire Wire Line
-	3200 4050 3200 3250
-Wire Wire Line
-	3050 4100 3050 3050
-Wire Wire Line
-	3050 3050 3200 3050
-Wire Wire Line
-	4350 4000 4350 3150
-Wire Wire Line
-	4350 3150 4000 3150
-Wire Wire Line
-	6850 2450 4200 2450
-Wire Wire Line
-	4200 2450 4200 3050
-Wire Wire Line
-	4200 3050 4000 3050
-Wire Wire Line
-	7350 1450 7350 3150
-Wire Wire Line
-	6700 1450 7350 1450
-Connection ~ 7100 1450
-Wire Wire Line
-	6500 1750 6500 1950
-Wire Wire Line
-	6000 1950 7700 1950
-Connection ~ 6500 1950
-Wire Wire Line
-	6300 1450 4850 1450
-Wire Wire Line
-	4850 1450 4850 2250
-Wire Wire Line
-	4500 2250 7800 2250
-Wire Wire Line
-	5500 1950 4700 1950
-Wire Wire Line
-	4700 1950 4700 3600
-Wire Wire Line
-	4700 3600 4650 3600
-Connection ~ 4650 3800
-Connection ~ 7100 1950
-Wire Wire Line
-	6750 2700 7250 2700
-Wire Wire Line
-	7250 2700 7250 2100
-Wire Wire Line
-	7250 2100 7600 2100
-Wire Wire Line
-	7600 2100 7600 1500
-Wire Wire Line
-	7600 1500 7700 1500
-Wire Wire Line
-	8950 1600 8950 1500
-Wire Wire Line
-	8950 1900 8950 1700
-Wire Wire Line
-	8950 1600 9150 1600
-Wire Wire Line
-	8950 1700 9150 1700
-Wire Wire Line
-	9150 1800 9000 1800
-Wire Wire Line
-	9000 1800 9000 2300
-Wire Wire Line
-	9000 2300 9150 2300
-Wire Wire Line
-	9150 1900 9150 2500
-Wire Wire Line
-	6750 2200 8350 2200
-Wire Wire Line
-	6750 2200 6750 2600
-Wire Wire Line
-	8300 2800 8450 2800
-Wire Wire Line
-	8350 2200 8350 2800
-Connection ~ 8350 2800
-Wire Wire Line
-	8950 2800 9150 2800
-Wire Wire Line
-	7800 2250 7800 2800
-Connection ~ 4850 2250
-Wire Wire Line
-	9150 3000 8950 3000
-Wire Wire Line
-	8450 4150 8450 3000
-Connection ~ 7350 4150
-Wire Wire Line
-	3200 3150 3150 3150
-Wire Wire Line
-	3150 3150 3150 4300
-Wire Wire Line
-	3150 4300 6900 4300
-Wire Wire Line
-	6900 4300 6900 3700
-Wire Wire Line
-	6900 3700 6750 3700
+	9300 3750 9300 3500
+Connection ~ 8450 4150
+Wire Wire Line
+	8800 2100 8800 3500
+Connection ~ 7600 2100
+$Comp
+L PN2222A Q1
+U 1 1 53121D07
+P 6500 1550
+F 0 "Q1" H 6500 1402 40  0000 R CNN
+F 1 "PN2222A" H 6500 1700 40  0000 R CNN
+F 2 "TO92" H 6400 1652 29  0000 C CNN
+F 3 "~" H 6500 1550 60  0000 C CNN
+	1    6500 1550
+	0    1    -1   0
+$EndComp
 $EndSCHEMATC
